Commit message: added gazebo materials

File: models/cengaver_core.xacro (robot description, xacro)
@@ -53,4 +53,7 @@
           </inertial>
     </link>
+    <gazebo reference="chassis">
+        <material>PR2/Grey1   </material>
+      </gazebo>
     <!-- FRONT LEFT WHEEL LINK -->
     <joint name="front_left_wheel_joint" type="continuous">
@@ -95,4 +98,7 @@
           </inertial>
     </link>
+    <gazebo reference="front_left_wheel">
+        <material>Gazebo/Red</material>
+      </gazebo>
     <!-- FRONT RIGHT WHEEL LINK -->
     <joint name="front_right_wheel_joint" type="continuous">
@@ -137,4 +143,7 @@
           </inertial>
     </link>
+    <gazebo reference="front_right_wheel">
+        <material>Gazebo/Red</material>
+      </gazebo>
     <!-- BACK LEFT WHEEL LINK -->
     <joint name="back_left_wheel_joint" type="continuous">
@@ -179,4 +188,7 @@
           </inertial>
     </link>
+    <gazebo reference="back_left_wheel">
+        <material>Gazebo/Black</material>
+      </gazebo>
     <!-- BACK RIGHT WHEEL LINK -->
     <joint name="back_right_wheel_joint" type="continuous">
@@ -221,3 +233,6 @@
           </inertial>
     </link>
+    <gazebo reference="back_right_wheel">
+        <material>Gazebo/Red</material>
+      </gazebo>
 </robot>
