Commit message: .

File: models/cengaver.urdf (robot description, URDF)
Before this commit: robot cengaver_rover, 9 links, 8 joints
Links:
- link back_left_wheel: geometry collision mesh filename=../meshes/wheel1.STL; visual mesh filename=../meshes/wheel1.STL
- link back_right_wheel: geometry collision mesh filename=../meshes/wheel1.STL; visual mesh filename=../meshes/wheel1.STL
- link chassis: geometry collision mesh filename=../meshes/base_link.STL; visual mesh filename=../meshes/base_link.STL
- link front_left_wheel: geometry collision mesh filename=../meshes/wheel1.STL; visual mesh filename=../meshes/wheel1.STL
- link front_right_wheel: geometry collision mesh filename=../meshes/wheel1.STL; visual mesh filename=../meshes/wheel1.STL

Commit message: Added base_footprint link and joint for slam_toolbox compatibility

File: models/cengaver.urdf (robot description, URDF)
Before this commit: robot cengaver_rover, 9 links, 8 joints
Links:
- added link base_footprint
Joints:
- added joint base_footprint_joint: type fixed, parent base_link, child base_footprint, origin xyz=0 0 0 rpy=0 0 0

File: models/cengaver_core.xacro (robot description, xacro)
@@ -15,4 +15,11 @@
     <link name="base_link">
     </link>
+    <joint name="base_footprint_joint" type="fixed">
+        <parent link="base_link"/>
+	    <child link="base_footprint"/>
+	    <origin xyz="0 0 0" rpy="0 0 0"/>
+    </joint>
+    <link name="base_footprint">
+    </link>
     <joint name="chassis_joint" type="fixed">
         <parent link="base_link" />
