Commit message: fixed lidar frame and camera joint position

File: models/camera.xacro (robot description, xacro)
@@ -1,8 +1,11 @@
 <?xml version="1.0"?>
 <robot xmlns:xacro="http://www.ros.org/wiki/xacro" >
+    <material name="red_camera">
+        <color rgba="1 0 0 1" />
+    </material>
     <joint name="camera_joint" type="fixed">
         <parent link="chassis"/>
         <child link="camera_link"/>
-        <origin xyz="0.305 0 0.08" rpy="0 0 0"/>
+        <origin xyz="0.205 0 0.08" rpy="0 0 0"/>
     </joint>
     <link name="camera_link">
@@ -11,5 +14,5 @@
                 <box size="0.010 0.03 0.03"/>
             </geometry>
-            <material name="red"/>
+            <material name="red_camera"/>
         </visual>
     </link>

File: models/lidar.xacro (robot description, xacro)
@@ -1,4 +1,7 @@
 <?xml version="1.0"?>
 <robot xmlns:xacro="http://www.ros.org/wiki/xacro" >
+    <material name="red_laser">
+        <color rgba="1 0 0 1" />
+    </material>
     <xacro:macro name="inertial_cylinder" params="mass radius length">
         <inertial>
@@ -11,5 +14,5 @@
         <parent link="chassis"/>
         <child link="laser_frame"/>
-        <origin xyz="0.1 0 0.175" rpy="0 0 0"/>
+        <origin xyz="0.1 0 0.175" rpy="0 0 ${pi}"/>
     </joint>
     <link name="laser_frame">
@@ -18,5 +21,5 @@
                 <cylinder radius="0.05" length="0.04"/>
             </geometry>
-            <material name="red"/>
+            <material name="red_laser"/>
         </visual>
         <collision>
@@ -41,6 +44,6 @@
                 </scan>
                 <range>
-                    <min>0.3</min>
-                    <max>12</max>
+                    <min>0.15</min>
+                    <max>6</max>
                 </range>
             </ray>

Commit message: added new launch file

File: models/camera.xacro (robot description, xacro)
@@ -16,4 +16,9 @@
             <material name="red_camera"/>
         </visual>
+        <colision>
+            <geometry>
+                <box size="0.010 0.03 0.03"/>
+            </geometry>
+        </colision>
     </link>
     <joint name="camera_optical_joint" type="fixed">
@@ -28,7 +33,7 @@
             <pose> 0 0 0 0 0 0 </pose>
             <visualize>true</visualize>
-            <update_rate>10</update_rate>
+            <update_rate>30</update_rate>
             <camera>
-                <horizontal_fov>1.089</horizontal_fov>
+                <horizontal_fov>1.256</horizontal_fov>
                 <image>
                     <format>R8G8B8</format>
@@ -38,5 +43,5 @@
                 <clip>
                     <near>0.05</near>
-                    <far>8.0</far>
+                    <far>20.0</far>
                 </clip>
             </camera>

File: models/gazebo_control.xacro (robot description, xacro)
@@ -27,6 +27,6 @@
             <wheel_diameter>${2*0.11736}</wheel_diameter>
             <!-- limits -->
-            <max_wheel_torque>500</max_wheel_torque>
-            <max_wheel_acceleration>2.0</max_wheel_acceleration>
+            <max_wheel_torque>1000</max_wheel_torque>
+            <max_wheel_acceleration>3.0</max_wheel_acceleration>
             <!-- Output -->
             <odometry_frame>odom</odometry_frame>
