Commit message: lidar model and imu

File: models/lidar.xacro (robot description, xacro)
@@ -3,4 +3,7 @@
     <material name="red_laser">
         <color rgba="1 0 0 1" />
+    </material>
+    <material name="black_lidar">
+        <color rgba="0 0 0 1" />
     </material>
     <xacro:macro name="inertial_cylinder" params="mass radius length">
@@ -14,29 +17,31 @@
         <parent link="chassis"/>
         <child link="laser_frame"/>
-        <origin xyz="0.1 0 0.175" rpy="0 0 ${pi}"/>
+        <origin xyz="0.14 0 0.175" rpy="0 0 ${pi}"/>
     </joint>
     <link name="laser_frame">
         <visual>
+            <origin xyz="0 0 -0.01" rpy="0 0 0"/>
             <geometry>
-                <cylinder radius="0.05" length="0.04"/>
+                <mesh filename="package://cengaver_rover_description/meshes/rplidar_a1.STL" />
             </geometry>
-            <material name="red_laser"/>
+            <material name="black_lidar"/>
         </visual>
         <collision>
+            <origin xyz="0 0 0" rpy="0 0 0"/>
             <geometry>
-                <cylinder radius="0.05" length="0.04"/>
+                <mesh filename="package://cengaver_rover_description/meshes/rplidar_a1.STL" />
             </geometry>
         </collision>
     </link>
     <gazebo reference="laser_frame">
-        <material>Gazebo/Red</material>
+        <material>Gazebo/Black</material>
         <sensor name="laser" type="ray">
             <pose> 0 0 0 0 0 0 </pose>
             <visualize>true</visualize>
-            <update_rate>10</update_rate>
+            <update_rate>5.5</update_rate>
             <ray>
                 <scan>
                     <horizontal>
-                        <samples>360</samples>
+                        <samples>363</samples>
                         <min_angle>-3.14</min_angle>
                         <max_angle>3.14</max_angle>

Commit message: fixed lidar collision

File: models/lidar.xacro (robot description, xacro)
@@ -28,5 +28,5 @@
         </visual>
         <collision>
-            <origin xyz="0 0 0" rpy="0 0 0"/>
+            <origin xyz="0 0 -0.01" rpy="0 0 0"/>
             <geometry>
                 <mesh filename="package://cengaver_rover_description/meshes/rplidar_a1.STL" />
