Commit message: changed package name to match repo

File: models/cengaver.urdf.xacro (robot description, xacro)
@@ -3,5 +3,5 @@
     <xacro:include filename="cengaver_core.xacro" />
     <xacro:include filename="gazebo_control.xacro"/>
-    <xacro:include filename="$(find cengaver_rover)/models/lidar.xacro" />
+    <xacro:include filename="$(find cengaver_rover_description)/models/lidar.xacro" />
     <xacro:include filename="camera.xacro" />
 </robot>

File: models/cengaver_core.xacro (robot description, xacro)
@@ -26,5 +26,5 @@
                 rpy="0 0 ${pi/2}" />
             <geometry>
-                <mesh filename="package://cengaver_rover/meshes/base_link.STL" />
+                <mesh filename="package://cengaver_rover_description/meshes/base_link.STL" />
             </geometry>
             <material name="chassis_material" />
@@ -35,5 +35,5 @@
                 rpy="0 0 ${pi/2}" />
             <geometry>
-                <mesh filename="package://cengaver_rover/meshes/base_link.STL" />
+                <mesh filename="package://cengaver_rover_description/meshes/base_link.STL" />
             </geometry>
         </collision>
@@ -71,5 +71,5 @@
                 rpy="0 0 0" />
             <geometry>
-                <mesh filename="package://cengaver_rover/meshes/wheel1.STL" />
+                <mesh filename="package://cengaver_rover_description/meshes/wheel1.STL" />
             </geometry>
             <material name="red_wheel_material" />
@@ -80,5 +80,5 @@
                 rpy="0 0 0" />
             <geometry>
-                <mesh filename="package://cengaver_rover/meshes/wheel1.STL" />
+                <mesh filename="package://cengaver_rover_description/meshes/wheel1.STL" />
             </geometry>
         </collision>
@@ -116,5 +116,5 @@
                 rpy="0 0 0" />
             <geometry>
-                <mesh filename="package://cengaver_rover/meshes/wheel1.STL" />
+                <mesh filename="package://cengaver_rover_description/meshes/wheel1.STL" />
             </geometry>
             <material name="red_wheel_material" />
@@ -125,5 +125,5 @@
                 rpy="0 0 0" />
             <geometry>
-                <mesh filename="package://cengaver_rover/meshes/wheel1.STL" />
+                <mesh filename="package://cengaver_rover_description/meshes/wheel1.STL" />
             </geometry>
         </collision>
@@ -161,5 +161,5 @@
                 rpy="0 0 0" />
             <geometry>
-                <mesh filename="package://cengaver_rover/meshes/wheel1.STL" />
+                <mesh filename="package://cengaver_rover_description/meshes/wheel1.STL" />
             </geometry>
             <material name="black_wheel_material" />
@@ -170,5 +170,5 @@
                 rpy="0 0 0" />
             <geometry>
-                <mesh filename="package://cengaver_rover/meshes/wheel1.STL" />
+                <mesh filename="package://cengaver_rover_description/meshes/wheel1.STL" />
             </geometry>
         </collision>
@@ -206,5 +206,5 @@
                 rpy="0 0 0" />
             <geometry>
-                <mesh filename="package://cengaver_rover/meshes/wheel1.STL" />
+                <mesh filename="package://cengaver_rover_description/meshes/wheel1.STL" />
             </geometry>
             <material name="red_wheel_material" />
@@ -215,5 +215,5 @@
                 rpy="0 0 0" />
             <geometry>
-                <mesh filename="package://cengaver_rover/meshes/wheel1.STL" />
+                <mesh filename="package://cengaver_rover_description/meshes/wheel1.STL" />
             </geometry>
         </collision>

Commit message: updated urdf files

File: models/cengaver.urdf.xacro (robot description, xacro)
@@ -5,3 +5,4 @@
     <xacro:include filename="$(find cengaver_rover_description)/models/lidar.xacro" />
     <xacro:include filename="$(find cengaver_rover_description)/models/camera.xacro" />
+    <xacro:include filename="$(find cengaver_rover_description)/models/imu.xacro" />
 </robot>

File: models/cengaver_core.xacro (robot description, xacro)
@@ -68,6 +68,6 @@
         <child link="front_left_wheel" />
         <origin
-            xyz="0.3379 ${0.27998 + 0.114} 0.11736"
-            rpy=" 0 -1.5708 -1.5708" />
+            xyz="0.338 0.394 0.117"
+            rpy=" 0 -1.571 -1.571" />
         <axis xyz="0 0 1" />
     </joint>
@@ -113,6 +113,6 @@
         <child link="front_right_wheel" />
         <origin
-            xyz="0.3379 ${-0.27998 - 0.114} 0.11736"
-            rpy=" 0 1.5708 -1.5708" />
+            xyz="0.338 -0.394 0.117"
+            rpy=" 0 1.571 -1.571" />
         <axis xyz="0 0 -1" />
     </joint>
@@ -158,6 +158,6 @@
         <child link="back_left_wheel" />
         <origin
-            xyz="-0.3379 ${0.27998 + 0.114} 0.11736"
-            rpy=" 0 -1.5708 -1.5708" />
+            xyz="-0.338 0.394 0.117"
+            rpy=" 0 -1.571 -1.571" />
         <axis xyz="0 0 1" />
     </joint>
@@ -203,6 +203,6 @@
         <child link="back_right_wheel" />
         <origin
-            xyz="-0.3379 ${-0.27998 - 0.114} 0.11736"
-            rpy=" 0 1.5708 -1.5708" />
+            xyz="-0.338 -0.394 0.117"
+            rpy=" 0 1.571 -1.571" />
         <axis xyz="0 0 -1" />
     </joint>

File: models/gazebo_control.xacro (robot description, xacro)
@@ -26,5 +26,5 @@
             <right_joint>front_right_wheel_joint</right_joint>
             <right_joint>back_right_wheel_joint</right_joint>
-            <wheel_separation>${(0.27998 + 0.114)*2}</wheel_separation>
+            <wheel_separation>${0.394*2}</wheel_separation>
             <wheel_diameter>${2*0.11736}</wheel_diameter>
             <!-- limits -->
@@ -34,5 +34,5 @@
             <odometry_frame>odom</odometry_frame>
             <robot_base_frame>base_link</robot_base_frame>
-            <odometry_source>0</odometry_source>
+            <odometry_source>1</odometry_source>
             <!-- Set to true to publish sensor_msgs/JointState on /joint_states for the wheel joints, defaults to false -->
             <publish_wheel_joint_state>true</publish_wheel_joint_state>

File: models/imu.xacro (robot description, xacro)
@@ -1,33 +1,33 @@
 <?xml version="1.0"?>
 <robot xmlns:xacro="http://www.ros.org/wiki/xacro">
-    <joint name="imu_joint" type="fixed">
-        <parent link="chassis"/>
-        <child link="imu_link"/>
-        <origin xyz="0 0 0" rpy="0 0 0"/>
-    </joint>
-    <link name="imu_link">
-    </link>
-    <gazebo reference="imu_link">
-        <gravity>true</gravity>
-        <sensor name="imu_sensor" type="imu">
-          <always_on>true</always_on>
-          <update_rate>100</update_rate>
-          <visualize>true</visualize>
-          <topic>__default_topic__</topic>
-          <plugin filename="libgazebo_ros_imu_sensor.so" name="imu_plugin">
-            <topicName>imu</topicName>
-            <bodyName>imu_link</bodyName>
-            <updateRateHZ>10.0</updateRateHZ>
-            <gaussianNoise>0.0</gaussianNoise>
-            <xyzOffset>0 0 0</xyzOffset>
-            <rpyOffset>0 0 0</rpyOffset>
-            <frameName>imu_link</frameName>
-            <initial_orientation_as_reference>false</initial_orientation_as_reference>
-            <ros>
-              <argument>~/out:=imu</argument>
-          </ros>
-          </plugin>
-          <pose>0 0 0 0 0 0</pose>
-        </sensor>
-      </gazebo>
+  <joint name="imu_joint" type="fixed">
+    <parent link="chassis" />
+    <child link="imu_link" />
+    <origin xyz="0 0 0" rpy="0 0 0" />
+  </joint>
+  <link name="imu_link">
+  </link>
+  <gazebo reference="imu_link">
+    <gravity>true</gravity>
+    <sensor name="imu_sensor" type="imu">
+      <always_on>true</always_on>
+      <update_rate>100</update_rate>
+      <visualize>true</visualize>
+      <topic>__default_topic__</topic>
+      <plugin filename="libgazebo_ros_imu_sensor.so" name="imu_plugin">
+        <ros>
+          <argument>~/out:=imu</argument>
+        </ros>
+        <topicName>imu</topicName>
+        <bodyName>imu_link</bodyName>
+        <updateRateHZ>10.0</updateRateHZ>
+        <gaussianNoise>0.0</gaussianNoise>
+        <xyzOffset>0 0 0</xyzOffset>
+        <rpyOffset>0 0 0</rpyOffset>
+        <frameName>imu_link</frameName>
+        <initialOrientationAsReference>false</initialOrientationAsReference>
+      </plugin>
+      <pose>0 0 0 0 0 0</pose>
+    </sensor>
+  </gazebo>
 </robot>

File: models/lidar.xacro (robot description, xacro)
@@ -51,5 +51,15 @@
                     <min>0.15</min>
                     <max>6</max>
+                    <resolution>0.05</resolution>
                 </range>
+                <noise>
+                    <type>gaussian</type>
+                    <!-- Noise parameters based on published spec for Hokuyo laser
+                         achieving "+-30mm" accuracy at range < 10m.  A mean of 0.0m and
+                         stddev of 0.01m will put 99.7% of samples within 0.03m of the true
+                         reading. -->
+                    <mean>0.0</mean>
+                    <stddev>0.005</stddev>
+                  </noise>
             </ray>
             <plugin name="laser_controller" filename="libgazebo_ros_ray_sensor.so">
